Commit message: estim of covers to urdf

File: spotmicro/util/pybullet_data/assets/urdf/spot.urdf (robot description, URDF)
Before this commit: robot rex, 23 links, 22 joints
Links:
- link front_left_leg_link_cover: mass None -> 0.03
- link front_right_leg_link_cover: mass None -> 0.03
- link rear_left_leg_link_cover: mass None -> 0.03
- link rear_right_leg_link_cover: mass None -> 0.03
