Commit message: merging from private repo

File: mini_ros/urdf/spot.urdf (robot description, URDF)
Before this commit: robot spot, 25 links, 24 joints
Links:
- removed link back
- removed link back_bracket
- removed link back_left_foot
- removed link back_left_hip
- removed link back_left_lower_leg
- removed link back_left_upper_leg
- removed link back_right_foot
- removed link back_right_hip
- removed link back_right_lower_leg
- removed link back_right_upper_leg
- removed link base_inertia
- removed link battery
- removed link chassis_left
- removed link chassis_right
- removed link front
- removed link front_bracket
- removed link front_left_foot
- removed link front_left_hip
- removed link front_left_lower_leg
- removed link front_left_upper_leg
- removed link front_right_foot
- removed link front_right_hip
- removed link front_right_lower_leg
- removed link front_right_upper_leg
- added link base_footprint
- added link chassis_front_link, mass 0.1; collision box size=0.058 0.11 0.07; visual mesh filename=package://mini_ros/stl/frontpart.stl scale=0.001 0.001 0.001
- added link chassis_rear_link, mass 0.1; collision box size=0.04 0.11 0.07; visual mesh filename=package://mini_ros/stl/backpart.stl scale=0.001 0.001 0.001
- added link front_left_foot_link, mass 0.1; collision box size=0.026 0.02 0.115; visual mesh filename=package://mini_ros/stl/lfoot.stl scale=0.001 0.001 0.001
- added link front_left_leg_link, mass 0.1; collision box size=0.028 0.036 0.12; visual mesh filename=package://mini_ros/stl/larm.stl scale=0.001 0.001 0.001
- added link front_left_leg_link_cover, mass 0.005; collision box size=0.028 0.036 0.12; visual mesh filename=package://mini_ros/stl/larm_cover.stl scale=0.001 0.001 0.001
- added link front_left_shoulder_link, mass 0.1; collision box size=0.044 0.038 0.07; visual mesh filename=package://mini_ros/stl/lshoulder.stl scale=0.001 0.001 0.001
- added link front_left_toe_link, mass 0.005; collision sphere radius=0.02; visual mesh filename=package://mini_ros/stl/foot.stl scale=0.001 0.001 0.001
- added link front_right_foot_link, mass 0.1; collision box size=0.026 0.02 0.115; visual mesh filename=package://mini_ros/stl/rfoot.stl scale=0.001 0.001 0.001
- added link front_right_leg_link, mass 0.1; collision box size=0.028 0.036 0.12; visual mesh filename=package://mini_ros/stl/rarm.stl scale=0.001 0.001 0.001
- added link front_right_leg_link_cover, mass 0.005; collision box size=0.028 0.036 0.12; visual mesh filename=package://mini_ros/stl/rarm_cover.stl scale=0.001 0.001 0.001
- added link front_right_shoulder_link, mass 0.1; collision box size=0.044 0.038 0.07; visual mesh filename=package://mini_ros/stl/rshoulder.stl scale=0.001 0.001 0.001
- added link front_right_toe_link, mass 0.005; collision sphere radius=0.02; visual mesh filename=package://mini_ros/stl/foot.stl scale=0.001 0.001 0.001
- added link rear_left_foot_link, mass 0.1; collision box size=0.026 0.02 0.115; visual mesh filename=package://mini_ros/stl/lfoot.stl scale=0.001 0.001 0.001
- added link rear_left_leg_link, mass 0.1; collision box size=0.028 0.036 0.12; visual mesh filename=package://mini_ros/stl/larm.stl scale=0.001 0.001 0.001
- added link rear_left_leg_link_cover, mass 0.005; collision box size=0.028 0.036 0.12; visual mesh filename=package://mini_ros/stl/larm_cover.stl scale=0.001 0.001 0.001
- added link rear_left_shoulder_link, mass 0.1; collision box size=0.044 0.038 0.07; visual mesh filename=package://mini_ros/stl/lshoulder.stl scale=0.001 0.001 0.001
- added link rear_left_toe_link, mass 0.005; collision sphere radius=0.02; visual mesh filename=package://mini_ros/stl/foot.stl scale=0.001 0.001 0.001
- added link rear_right_foot_link, mass 0.15; collision box size=0.026 0.02 0.115; visual mesh filename=package://mini_ros/stl/rfoot.stl scale=0.001 0.001 0.001
- added link rear_right_leg_link, mass 0.1; collision box size=0.028 0.036 0.12; visual mesh filename=package://mini_ros/stl/rarm.stl scale=0.001 0.001 0.001
- added link rear_right_leg_link_cover, mass 0.005; collision box size=0.028 0.036 0.12; visual mesh filename=package://mini_ros/stl/rarm_cover.stl scale=0.001 0.001 0.001
- added link rear_right_shoulder_link, mass 0.1; collision box size=0.044 0.038 0.07; visual mesh filename=package://mini_ros/stl/rshoulder.stl scale=0.001 0.001 0.001
- added link rear_right_toe_link, mass 0.005; collision sphere radius=0.02; visual mesh filename=package://mini_ros/stl/foot.stl scale=0.001 0.001 0.001
- link base_link: mass None -> 1.2; geometry collision box size=0.14 0.11 0.07; visual mesh filename=package://mini_ros/stl/mainbody.stl scale=0.001 0.001 0.001
Joints:
- removed joint back_left_leg_foot
- removed joint back_right_leg_foot
- removed joint base_back
- removed joint base_back_bracket
- removed joint base_battery
- removed joint base_front
- removed joint base_front_bracket
- removed joint base_left
- removed joint base_right
- removed joint front_left_leg_foot
- removed joint front_right_leg_foot
- removed joint motor_back_left_hip
- removed joint motor_back_left_lower_leg
- removed joint motor_back_left_upper_leg
- removed joint motor_back_right_hip
- removed joint motor_back_right_lower_leg
- removed joint motor_back_right_upper_leg
- removed joint motor_front_left_hip
- removed joint motor_front_left_lower_leg
- removed joint motor_front_left_upper_leg
- removed joint motor_front_right_hip
- removed joint motor_front_right_lower_leg
- removed joint motor_front_right_upper_leg
- added joint chassis_base_front: type fixed, parent base_link, child chassis_front_link, origin xyz=0 0 0 rpy=0 0 0
- added joint chassis_base_rear: type fixed, parent base_link, child chassis_rear_link, origin xyz=0 0 0 rpy=0 0 0
- added joint foot_motor_front_left: type revolute, parent front_left_leg_link, child front_left_foot_link, origin xyz=-0.01 0 -0.12 rpy=0 0 0, axis 0 1 0, limit lower=-0.1 upper=2.59 effort=3.5 velocity=9.5
- added joint foot_motor_front_right: type revolute, parent front_right_leg_link, child front_right_foot_link, origin xyz=-0.01 0 -0.12 rpy=0 0 0, axis 0 1 0, limit lower=-0.1 upper=2.59 effort=3.5 velocity=9.5
- added joint foot_motor_rear_left: type revolute, parent rear_left_leg_link, child rear_left_foot_link, origin xyz=-0.01 0 -0.12 rpy=0 0 0, axis 0 1 0, limit lower=-0.1 upper=2.59 effort=3.5 velocity=9.5
- added joint foot_motor_rear_right: type revolute, parent rear_right_leg_link, child rear_right_foot_link, origin xyz=-0.01 0 -0.12 rpy=0 0 0, axis 0 1 0, limit lower=-0.1 upper=2.59 effort=3.5 velocity=9.5
- added joint front_left_leg_cover_joint: type fixed, parent front_left_leg_link, child front_left_leg_link_cover, origin xyz=0 0 0 rpy=0 0 0
- added joint front_left_toe: type fixed, parent front_left_foot_link, child front_left_toe_link, origin xyz=0 0 -0.115 rpy=0 0 0
- added joint front_right_leg_cover_joint: type fixed, parent front_right_leg_link, child front_right_leg_link_cover, origin xyz=0 0 0 rpy=0 0 0
- added joint front_right_toe: type fixed, parent front_right_foot_link, child front_right_toe_link, origin xyz=0 0 -0.115 rpy=0 0 0
- added joint motor_front_left_leg: type revolute, parent front_left_shoulder_link, child front_left_leg_link, origin xyz=0 -0.052 0 rpy=0 0 0, axis 0 1 0, limit lower=-2.17 upper=0.97 effort=3.5 velocity=9.5
- added joint motor_front_left_shoulder: type revolute, parent base_link, child front_left_shoulder_link, origin xyz=-0.093 -0.036 0 rpy=0 0 0, axis 1 0 0, limit lower=-1.0 upper=1.0 effort=3.5 velocity=9.5
- added joint motor_front_right_leg: type revolute, parent front_right_shoulder_link, child front_right_leg_link, origin xyz=0 0.052 0 rpy=0 0 0, axis 0 1 0, limit lower=-2.17 upper=0.97 effort=3.5 velocity=9.5
- added joint motor_front_right_shoulder: type revolute, parent base_link, child front_right_shoulder_link, origin xyz=-0.093 0.036 0 rpy=0 0 0, axis 1 0 0, limit lower=-1.0 upper=1.0 effort=3.5 velocity=9.5
- added joint motor_rear_left_leg: type revolute, parent rear_left_shoulder_link, child rear_left_leg_link, origin xyz=0 -0.052 0 rpy=0 0 0, axis 0 1 0, limit lower=-2.17 upper=0.97 effort=3.5 velocity=9.5
- added joint motor_rear_left_shoulder: type revolute, parent base_link, child rear_left_shoulder_link, origin xyz=0.093 -0.036 0 rpy=0 0 0, axis 1 0 0, limit lower=-1.0 upper=1.0 effort=3.5 velocity=9.5
- added joint motor_rear_right_leg: type revolute, parent rear_right_shoulder_link, child rear_right_leg_link, origin xyz=0 0.052 0 rpy=0 0 0, axis 0 1 0, limit lower=-2.17 upper=0.97 effort=3.5 velocity=9.5
- added joint motor_rear_right_shoulder: type revolute, parent base_link, child rear_right_shoulder_link, origin xyz=0.093 0.036 0 rpy=0 0 0, axis 1 0 0, limit lower=-1.0 upper=1.0 effort=3.5 velocity=9.5
- added joint rear_left_leg_cover_joint: type fixed, parent rear_left_leg_link, child rear_left_leg_link_cover, origin xyz=0 0 0 rpy=0 0 0
- added joint rear_left_toe: type fixed, parent rear_left_foot_link, child rear_left_toe_link, origin xyz=0 0 -0.115 rpy=0 0 0
- added joint rear_right_leg_cover_joint: type fixed, parent rear_right_leg_link, child rear_right_leg_link_cover, origin xyz=0 0 0 rpy=0 0 0
- added joint rear_right_toe: type fixed, parent rear_right_foot_link, child rear_right_toe_link, origin xyz=0 0 -0.115 rpy=0 0 0
- joint base_base: child base_inertia -> base_link; parent base_link -> base_footprint
