Commit message: merging from private repo

File: mini_ros/urdf/spot.urdf.xacro (robot description, xacro)
@@ -3,467 +3,459 @@
   <!-- Include Macros -->
   <xacro:include filename="$(find mini_ros)/urdf/spot_macro.xacro" />
-  <xacro:include filename="$(find mini_ros)/urdf/transmissions.xacro" />
-  <!-- <xacro:include filename="$(find mini_ros)/urdf/accessories.urdf.xacro" /> -->
   <!-- Robot description -->
-  <!-- STATIC Links -->
-  <link name="base_link"/>
+  <!-- Links -->
+  <link name="base_footprint"/>
   <!-- MAIN BODY -->
-  <xacro:mesh_link name="base_inertia"
-              origin_rpy="0 0 ${pi/2}" origin_xyz="-0.16 0.035 -0.045"
-              i_rpy="0 0 0" i_xyz="0 0 0"
-              mass="0.6"
-              c_xyz="0 0 0"
-              length="0.114"
-              width="0.2"
-              height="0.1"
-              matname="orange"
-              meshfile="package://mini_ros/stl/OpenQuadruped/MAINBODY.stl"
-              meshscale="1 1 1" /> <!-- m to mm -->
-  <!-- BATTERY -->
-  <xacro:mesh_link name="battery"
-              origin_rpy="0 0 ${pi/2}" origin_xyz="-0.15 0.035 -0.022"
-              i_rpy="0 0 0" i_xyz="0 0 0"
-              mass="0.4"
-              c_xyz="0 0 0"
-              length="0.048"
-              width="0.145"
-              height="0.026"
-              matname="black"
-              meshfile="package://mini_ros/stl/OpenQuadruped/Battery.stl"
-              meshscale="1 1 1" /> <!-- m to mm -->
-  <!-- CHASSIS LEFT -->
-  <xacro:mesh_link name="chassis_left"
-              origin_rpy="0 ${pi/2} -${pi/2}" origin_xyz="0.016 0.003 0"
-              i_rpy="0 0 0" i_xyz="0 0 0"
-              mass="0.01"
-              c_xyz="0 0 0"
-              length="0.06"
-              width="0.15"
-              height="0.006"
-              matname="black"
-              meshfile="package://mini_ros/stl/OpenQuadruped/Chassis_Left_Side.stl"
-              meshscale="1 1 1" /> <!-- m to mm -->
-  <!-- CHASSIS Right -->
-  <xacro:mesh_link name="chassis_right"
-              origin_rpy="0 ${pi/2} ${pi/2}" origin_xyz="-0.016 -0.003 0"
-              i_rpy="0 0 0" i_xyz="0 0 0"
-              mass="0.01"
-              c_xyz="0 0 0"
-              length="0.06"
-              width="0.15"
-              height="0.006"
-              matname="black"
-              meshfile="package://mini_ros/stl/OpenQuadruped/Chassis_Right_Side.stl"
-              meshscale="1 1 1" /> <!-- m to mm -->
-  <!-- FRONT -->
-  <xacro:mesh_link name="front"
-              origin_rpy="0 0 ${pi/2}" origin_xyz="-0.16 0.035 -0.045"
-              i_rpy="0 0 0" i_xyz="0 0 0"
-              mass="0.1"
-              c_xyz="0.16 0 0.006"
-              length="0.114"
-              width="0.045"
-              height="0.085"
-              matname="orange"
-              meshfile="package://mini_ros/stl/OpenQuadruped/Front.stl"
-              meshscale="1 1 1" /> <!-- m to mm -->
-  <!-- BACK -->
-  <xacro:mesh_link name="back"
-              origin_rpy="0 0 ${pi/2}" origin_xyz="-0.16 0.035 -0.045"
-              i_rpy="0 0 0" i_xyz="0 0 0"
-              mass="0.1"
-              c_xyz="-0.16 0 0.006"
-              length="0.114"
-              width="0.075"
-              height="0.085"
-              matname="orange"
-              meshfile="package://mini_ros/stl/OpenQuadruped/Back.stl"
-              meshscale="1 1 1" /> <!-- m to mm -->
-  <!-- FRONT BRACKET -->
-  <xacro:mesh_link name="front_bracket"
-              origin_rpy="0 0 ${pi/2}" origin_xyz="-0.16 0.035 -0.045"
-              i_rpy="0 0 0" i_xyz="0 0 0"
-              mass="0.1"
-              c_xyz="0.1 0 0"
-              length="0.025"
-              width="0.075"
-              height="0.085"
-              matname="black"
-              meshfile="package://mini_ros/stl/OpenQuadruped/Front_Bracket.stl"
-              meshscale="1 1 1" /> <!-- m to mm -->
-  <!-- BACK BRACKET -->
-  <xacro:mesh_link name="back_bracket"
-              origin_rpy="0 0 ${pi/2}" origin_xyz="-0.16 0.035 -0.045"
-              i_rpy="0 0 0" i_xyz="0 0 0"
-              mass="0.1"
-              c_xyz="-0.1 0 0"
-              length="0.025"
-              width="0.075"
-              height="0.085"
-              matname="black"
-              meshfile="package://mini_ros/stl/OpenQuadruped/Back_Bracket.stl"
-              meshscale="1 1 1" /> <!-- m to mm -->
-  <!-- DYNAMIC LINKS (Joints Included) -->
+  <xacro:mesh_link name="base_link"
+              origin_rpy="0 0 0" origin_xyz="-0.045 -0.060 -0.015"
+              i_rpy="0 0 0" i_xyz="0 0 0"
+              mass="1.2"
+              c_xyz="0 0 0"
+              length="0.14"
+              width="0.11"
+              height="0.07"
+              matname="black"
+              meshfile="package://mini_ros/stl/mainbody.stl"
+              meshscale="0.001 0.001 0.001" /> <!-- m to mm -->
+  <!-- HEAD -->
+  <xacro:mesh_link name="chassis_front_link"
+              origin_rpy="0 0 0" origin_xyz="-0.040 -0.060 -0.0140"
+              i_rpy="0 0 0" i_xyz="-0.145 0 0"
+              mass="0.1"
+              c_xyz="-0.145 0 0"
+              length="0.058"
+              width="0.11"
+              height="0.07"
+              matname="yellow"
+              meshfile="package://mini_ros/stl/frontpart.stl"
+              meshscale="0.001 0.001 0.001" />
+  <!-- TAIL -->
+  <xacro:mesh_link name="chassis_rear_link"
+              origin_rpy="0 0 0" origin_xyz="-0.040 -0.060 -0.0140"
+              i_rpy="0 0 0" i_xyz="0.135 0 0"
+              mass="0.1"
+              c_xyz="0.135 0 0"
+              length="0.04"
+              width="0.11"
+              height="0.07"
+              matname="yellow"
+              meshfile="package://mini_ros/stl/backpart.stl"
+              meshscale="0.001 0.001 0.001" />
   <!-- FRONT LEFT LEG -->
-  <!-- HIP -->
-  <xacro:mesh_link name="front_left_hip"
-              origin_rpy="0 0 ${pi/2}" origin_xyz="-0.25 -0.0044 -0.067"
-              i_rpy="0 0 0" i_xyz="0 0.075 0"
-              mass="0.2"
-              c_xyz="0.015 0.01 -0.01"
-              length="0.05"
-              width="0.065"
-              height="0.065"
-              matname="black"
-              meshfile="package://mini_ros/stl/OpenQuadruped/LEFT_HIP.stl"
-              meshscale="1 1 1" /> <!-- m to mm -->
-  <xacro:rev_joint name="motor_front_left_hip" type="revolute"
+  <!-- SHOULDER -->
+  <xacro:mesh_link name="front_left_shoulder_link"
+              origin_rpy="0 0 0" origin_xyz="-0.135 -0.02 -0.01"
+              i_rpy="0 0 0" i_xyz="0 0 0"
+              mass="0.1"
+              c_xyz="0 0 0"
+              length="0.044"
+              width="0.038"
+              height="0.07"
+              matname="black"
+              meshfile="package://mini_ros/stl/lshoulder.stl"
+              meshscale="0.001 0.001 0.001" />
+  <!-- COVER -->
+  <xacro:mesh_link name="front_left_leg_link_cover"
+              origin_rpy="0 0 0" origin_xyz="-0.125 0.04 -0.02"
+              i_rpy="0 0 0" i_xyz="0.0 0.0 -0.050"
+              mass="0.005"
+              c_xyz="0.0 0.0 -0.050"
+              length="0.028"
+              width="0.036"
+              height="0.12"
+              matname="yellow"
+              meshfile="package://mini_ros/stl/larm_cover.stl"
+              meshscale="0.001 0.001 0.001" />
+  <!-- LEG -->
+  <xacro:mesh_link name="front_left_leg_link"
+              origin_rpy="0 0 0" origin_xyz="-0.125 0.04 -0.02"
+              i_rpy="0 0 0" i_xyz="0.0 0.0 -0.050"
+              mass="0.1"
+              c_xyz="0.0 0.0 -0.050"
+              length="0.028"
+              width="0.036"
+              height="0.12"
+              matname="black"
+              meshfile="package://mini_ros/stl/larm.stl"
+              meshscale="0.001 0.001 0.001" />
+  <!-- FOOT -->
+  <xacro:mesh_link name="front_left_foot_link"
+              origin_rpy="0 0 0" origin_xyz="-0.120 0.04 0.1"
+              i_rpy="0 0 0" i_xyz="0.0 0.0 -0.050"
+              mass="0.1"
+              c_xyz="0.0 0.0 -0.050"
+              length="0.026"
+              width="0.02"
+              height="0.115"
+              matname="black"
+              meshfile="package://mini_ros/stl/lfoot.stl"
+              meshscale="0.001 0.001 0.001" />
+<!-- TOE -->
+  <xacro:mesh_link_sphere name="front_left_toe_link"
+              origin_rpy="0 -0.40010 0" origin_xyz="0 -0.01 0"
+              i_rpy="0 0 0" i_xyz="0 0 0"
+              mass="0.005"
+              c_xyz="0 0 0"
+              length="0.02"
+              width="0.02"
+              height="0.02"
+              radius="0.02"
+              matname="grey"
+              meshfile="package://mini_ros/stl/foot.stl"
+              meshscale="0.001 0.001 0.001" />
+  <!-- FRONT RIGHT LEG -->
+  <!-- SHOULDER -->
+  <xacro:mesh_link name="front_right_shoulder_link"
+              origin_rpy="0 0 0" origin_xyz="-0.135 -0.09 -0.01"
+              i_rpy="0 0 0" i_xyz="0 0 0"
+              mass="0.1"
+              c_xyz="0 0 0"
+              length="0.044"
+              width="0.038"
+              height="0.07"
+              matname="black"
+              meshfile="package://mini_ros/stl/rshoulder.stl"
+              meshscale="0.001 0.001 0.001" />
+  <!-- COVER -->
+  <xacro:mesh_link name="front_right_leg_link_cover"
+              origin_rpy="0 0 0" origin_xyz="-0.125 -0.15 -0.02"
+              i_rpy="0 0 0" i_xyz="0.0 0.0 -0.050"
+              mass="0.005"
+              c_xyz="0.0 0.0 -0.050"
+              length="0.028"
+              width="0.036"
+              height="0.12"
+              matname="yellow"
+              meshfile="package://mini_ros/stl/rarm_cover.stl"
+              meshscale="0.001 0.001 0.001" />
+  <!-- LEG -->
+  <xacro:mesh_link name="front_right_leg_link"
+              origin_rpy="0 0 0" origin_xyz="-0.125 -0.15 -0.02"
+              i_rpy="0 0 0" i_xyz="0.0 0.0 -0.050"
+              mass="0.1"
+              c_xyz="0.0 0.0 -0.050"
+              length="0.028"
+              width="0.036"
+              height="0.12"
+              matname="black"
+              meshfile="package://mini_ros/stl/rarm.stl"
+              meshscale="0.001 0.001 0.001" />
+  <!-- FOOT -->
+  <xacro:mesh_link name="front_right_foot_link"
+              origin_rpy="0 0 0" origin_xyz="-0.120 -0.15 0.1"
+              i_rpy="0 0 0" i_xyz="0.0 0.0 -0.050"
+              mass="0.1"
+              c_xyz="0.0 0.0 -0.050"
+              length="0.026"
+              width="0.02"
+              height="0.115"
+              matname="black"
+              meshfile="package://mini_ros/stl/rfoot.stl"
+              meshscale="0.001 0.001 0.001" />
+<!-- TOE -->
+  <xacro:mesh_link_sphere name="front_right_toe_link"
+              origin_rpy="0 -0.40010 0" origin_xyz="0 -0.01 0"
+              i_rpy="0 0 0" i_xyz="0 0 0"
+              mass="0.005"
+              c_xyz="0 0 0"
+              length="0.02"
+              width="0.02"
+              height="0.02"
+              radius="0.02"
+              matname="grey"
+              meshfile="package://mini_ros/stl/foot.stl"
+              meshscale="0.001 0.001 0.001" />
+  <!-- REAR LEFT LEG -->
+  <!-- SHOULDER -->
+  <xacro:mesh_link name="rear_left_shoulder_link"
+              origin_rpy="0 0 0" origin_xyz="-0.135 -0.02 -0.01"
+              i_rpy="0 0 0" i_xyz="0 0 0"
+              mass="0.1"
+              c_xyz="0 0 0"
+              length="0.044"
+              width="0.038"
+              height="0.07"
+              matname="black"
+              meshfile="package://mini_ros/stl/lshoulder.stl"
+              meshscale="0.001 0.001 0.001" />
+  <!-- COVER -->
+  <xacro:mesh_link name="rear_left_leg_link_cover"
+              origin_rpy="0 0 0" origin_xyz="-0.125 0.04 -0.02"
+              i_rpy="0 0 0" i_xyz="0.0 0.0 -0.050"
+              mass="0.005"
+              c_xyz="0.0 0.0 -0.050"
+              length="0.028"
+              width="0.036"
+              height="0.12"
+              matname="yellow"
+              meshfile="package://mini_ros/stl/larm_cover.stl"
+              meshscale="0.001 0.001 0.001" />
+  <!-- LEG -->
+  <xacro:mesh_link name="rear_left_leg_link"
+              origin_rpy="0 0 0" origin_xyz="-0.125 0.04 -0.02"
+              i_rpy="0 0 0" i_xyz="0.0 0.0 -0.050"
+              mass="0.1"
+              c_xyz="0.0 0.0 -0.050"
+              length="0.028"
+              width="0.036"
+              height="0.12"
+              matname="black"
+              meshfile="package://mini_ros/stl/larm.stl"
+              meshscale="0.001 0.001 0.001" />
+  <!-- FOOT -->
+  <xacro:mesh_link name="rear_left_foot_link"
+              origin_rpy="0 0 0" origin_xyz="-0.120 0.04 0.1"
+              i_rpy="0 0 0" i_xyz="0.0 0.0 -0.050"
+              mass="0.1"
+              c_xyz="0.0 0.0 -0.050"
+              length="0.026"
+              width="0.02"
+              height="0.115"
+              matname="black"
+              meshfile="package://mini_ros/stl/lfoot.stl"
+              meshscale="0.001 0.001 0.001" />
+<!-- TOE -->
+  <xacro:mesh_link_sphere name="rear_left_toe_link"
+              origin_rpy="0 -0.40010 0" origin_xyz="0 -0.01 0"
+              i_rpy="0 0 0" i_xyz="0 0 0"
+              mass="0.005"
+              c_xyz="0 0 0"
+              length="0.02"
+              width="0.02"
+              height="0.02"
+              radius="0.02"
+              matname="grey"
+              meshfile="package://mini_ros/stl/foot.stl"
+              meshscale="0.001 0.001 0.001" />
+  <!-- REAR RIGHT LEG -->
+  <!-- SHOULDER -->
+  <xacro:mesh_link name="rear_right_shoulder_link"
+              origin_rpy="0 0 0" origin_xyz="-0.135 -0.09 -0.01"
+              i_rpy="0 0 0" i_xyz="0 0 0"
+              mass="0.1"
+              c_xyz="0 0 0"
+              length="0.044"
+              width="0.038"
+              height="0.07"
+              matname="black"
+              meshfile="package://mini_ros/stl/rshoulder.stl"
+              meshscale="0.001 0.001 0.001" />
+  <!-- COVER -->
+  <xacro:mesh_link name="rear_right_leg_link_cover"
+              origin_rpy="0 0 0" origin_xyz="-0.125 -0.15 -0.02"
+              i_rpy="0 0 0" i_xyz="0.0 0.0 -0.050"
+              mass="0.005"
+              c_xyz="0.0 0.0 -0.050"
+              length="0.028"
+              width="0.036"
+              height="0.12"
+              matname="yellow"
+              meshfile="package://mini_ros/stl/rarm_cover.stl"
+              meshscale="0.001 0.001 0.001" />
+  <!-- LEG -->
+  <xacro:mesh_link name="rear_right_leg_link"
+              origin_rpy="0 0 0" origin_xyz="-0.125 -0.15 -0.02"
+              i_rpy="0 0 0" i_xyz="0.0 0.0 -0.050"
+              mass="0.1"
+              c_xyz="0.0 0.0 -0.050"
+              length="0.028"
+              width="0.036"
+              height="0.12"
+              matname="black"
+              meshfile="package://mini_ros/stl/rarm.stl"
+              meshscale="0.001 0.001 0.001" />
+  <!-- FOOT -->
+  <xacro:mesh_link name="rear_right_foot_link"
+              origin_rpy="0 0 0" origin_xyz="-0.120 -0.15 0.1"
+              i_rpy="0 0 0" i_xyz="0.0 0.0 -0.050"
+              mass="0.15"
+              c_xyz="0.0 0.0 -0.050"
+              length="0.026"
+              width="0.02"
+              height="0.115"
+              matname="black"
+              meshfile="package://mini_ros/stl/rfoot.stl"
+              meshscale="0.001 0.001 0.001" />
+<!-- TOE -->
+  <xacro:mesh_link_sphere name="rear_right_toe_link"
+              origin_rpy="0 -0.40010 0" origin_xyz="0 -0.01 0"
+              i_rpy="0 0 0" i_xyz="0 0 0"
+              mass="0.005"
+              c_xyz="0 0 0"
+              length="0.02"
+              width="0.02"
+              height="0.02"
+              radius="0.02"
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
File: mini_ros/urdf/spot_macro.xacro (robot description, xacro)
@@ -1,6 +1,6 @@
 <?xml version="1.0" ?>
 <robot xmlns:xacro="http://www.ros.org/wiki/xacro">
-  <material name="orange">
-    <color rgba="1.0 0.5 0.0 1"/>
+  <material name="yellow">
+    <color rgba="0.92 0.83 0.0 1"/>
   </material>
   <material name="black">
@@ -48,12 +48,4 @@
       </inertial>
     </link>
-    <gazebo reference="${name}">
-        <xacro:if value="${matname == 'black'}">
-          <material>Gazebo/Black</material>
-        </xacro:if>
-        <xacro:if value="${matname == 'orange'}">
-          <material>Gazebo/Orange</material>
-        </xacro:if>
-    </gazebo>
   </xacro:macro>
   <xacro:macro name="mesh_link_sphere" params="name origin_xyz origin_rpy meshfile meshscale c_xyz matname mass i_xyz i_rpy length width height radius">
@@ -69,5 +61,5 @@
         <origin rpy="${origin_rpy}" xyz="${c_xyz}" />
         <geometry>
-          <mesh filename="${meshfile}" scale="${meshscale}"/>
+          <sphere radius="${radius}"/>
         </geometry>
         <contact_coefficients mu="10.1"/>
@@ -79,37 +71,4 @@
       </inertial>
     </link>
-    <gazebo reference="${name}">
-      <kp>1000000.0</kp>
-      <kd>1.0</kd>
-      <mu1>0.8</mu1>
-      <mu2>0.8</mu2>
-      <maxVel>0.0</maxVel>
-      <minDepth>0.001</minDepth>
-      <material>Gazebo/Orange</material>
-    </gazebo>
   </xacro:macro>
-  <!-- Left Leg: prefix is front or rear -->
-<!--   <xacro:macro name="LeftLeg" params="prefix reflect">
-    <link name="${prefix}_Left_Leg">
-        <visual>
-            <geometry>
-                <box size="${leglen} 0.1 0.2"/>
-            </geometry>
-            <origin xyz="0 0 -${leglen/2}" rpy="0 ${pi/2} 0"/>
-            <material name="white"/>
-        </visual>
-        <collision>
-            <geometry>
-                <box size="${leglen} 0.1 0.2"/>
-            </geometry>
-            <origin xyz="0 0 -${leglen/2}" rpy="0 ${pi/2} 0"/>
-        </collision>
-        <xacro:default_inertial mass="10"/>
-    </link>
-    <joint name="base_to_${prefix}_leg" type="fixed">
-        <parent link="base_link"/>
-        <child link="${prefix}_leg"/>
-        <origin xyz="0 ${reflect*(width+.02)} 0.25" />
-    </joint>
-</xacro:macro> -->
 </robot>
